File: cho-corne-ice/pcb/cho-corne-ice.kicad_pcb (KiCad board)
At the start: 2 copper layers, 275.5 x 105.6 mm, 121 parts, among them J1 BAT, J2 nice!view, J3 BAT, J4 nice!view, SW1 SW_PUSH, SW10 SW_PUSH, SW11 SW_PUSH, SW12 SW_PUSH, SW13 SW_PUSH, SW14 SW_PUSH, SW15 SW_PUSH, SW16 SW_PUSH, SW17 SW_PUSH, SW18 SW_PUSH, SW19 SW_PUSH, SW2 SW_PUSH, SW20 SW_PUSH, SW21 SW_PUSH, SW22 SW_PUSH, SW23 SW_PUSH, SW24 SW_PUSH, SW25 SW_PUSH, SW26 SW_PUSH, SW27 SW_PUSH, SW28 SW_PUSH, SW29 SW_PUSH, SW3 SW_PUSH, SW30 SW_PUSH, SW31 SW_PUSH, SW32 SW_PUSH, SW33 SW_PUSH, SW34 SW_PUSH, SW35 SW_PUSH, SW36 SW_PUSH, SW37 SW_PUSH, SW38 SW_PUSH, SW39 SW_PUSH, SW4 SW_PUSH, SW40 SW_PUSH, SW41 SW_PUSH, SW42 SW_PUSH, SW5 SW_PUSH, SW6 SW_PUSH, SW7 SW_PUSH, SW8 SW_PUSH, SW9 SW_PUSH, U1 nice_nano, U2 nice_nano

Commit message: revert reset switches
Parts:
- RSW1, RSW2: footprint keeblib:alps_sksn -> kbd:ResetSW_1side
- moved RSW1 1.55 mm to (143.3, 66.5)
- moved RSW2 1.32 mm to (153.5, 66.7)
Changed lines of the file:
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@@
   (net 97 "CS_r")
   (net 98 "unconnected-(U2-Pad2)")
-  (footprint "keeblib:alps_sksn" (layer "F.Cu")
-    (at 144.8495 66.541 90)
+  (footprint "kbd:ResetSW_1side" (layer "F.Cu")
+    (at 143.2975 66.541 90)
     (property "Sheetfile" "File: cho-corne-ice.kicad_sch")
     (property "Sheetname" "")
     (attr through_hole)
-    (fp_text reference "RSW1" (at 0 -0.79 90) (layer "F.SilkS")
+    (fp_text reference "RSW1" (at 0 2.55 90) (layer "F.SilkS") hide
       (effects (font (size 1 1) (thickness 0.15)))
     )
-    (fp_text value "SW_PUSH" (at 0 -0.5 90) (layer "F.Fab") hide
+    (fp_text value "SW_PUSH" (at 0 -2.55 90) (layer "F.Fab")
       (effects (font (size 1 1) (thickness 0.15)))
     )
-    (fp_line (start 2.55 -1.65) (end 2.55 0) (layer "B.Fab") (width 0.12))
-    (fp_line (start -2.55 -1.65) (end 2.55 -1.65) (layer "B.Fab") (width 0.12))
-    (fp_line (start -2.55 0) (end -2.55 -1.65) (layer "B.Fab") (width 0.12))
-    (pad "" smd rect locked (at 3.2 -0.85 90) (size 0.6 0.8) (layers "F.Cu" "F.Paste" "F.Mask"))
-    (pad "" smd rect locked (at -3.2 -0.85 90) (size 0.6 0.8) (layers "F.Cu" "F.Paste" "F.Mask"))
-    (pad "1" smd rect locked (at 2.275 -2.575 90) (size 1.45 1.05) (layers "F.Cu" "F.Paste" "F.Mask")
+    (fp_text user "RESET" (at 0 0 90) (layer "F.SilkS")
+      (effects (font (size 1 1) (thickness 0.15)))
+    )
+    (fp_line (start -2.85 1.6) (end 2.85 1.6) (layer "F.SilkS") (width 0.15))
+    (fp_line (start -2.85 -1.6) (end -2.85 -1.35) (layer "F.SilkS") (width 0.15))
+    (fp_line (start -2.85 1.6) (end -2.85 1.35) (layer "F.SilkS") (width 0.15))
+    (fp_line (start -2.85 -1.6) (end 2.85 -1.6) (layer "F.SilkS") (width 0.15))
+    (fp_line (start 2.85 1.6) (end 2.85 1.35) (layer "F.SilkS") (width 0.15))
+    (fp_line (start 2.85 -1.6) (end 2.85 -1.35) (layer "F.SilkS") (width 0.15))
+    (pad "1" thru_hole circle locked (at 3.25 0 90) (size 2 2) (drill 1.3) (layers *.Cu "B.Mask")
       (net 35 "reset") (pinfunction "1") (pintype "passive"))
-    (pad "2" smd rect locked (at -2.275 -2.575 90) (size 1.45 1.05) (layers "F.Cu" "F.Paste" "F.Mask")
+    (pad "2" thru_hole circle locked (at -3.25 0 90) (size 2 2) (drill 1.3) (layers *.Cu "B.Mask")
       (net 26 "GND") (pinfunction "2") (pintype "passive"))
-    (model "C:/Users/cwiggins/Downloads/keyboards/keeblib.pretty/3d/3Dâéâfâï_SKSNL.STEP"
-      (offset (xyz 0 2 0))
+    (model "/Users/foostan/src/github.com/foostan/kbd/kicad-packages3D/kbd.3dshapes/tact-switch.step"
+      (offset (xyz 0 0 3.47))
       (scale (xyz 1 1 1))
       (rotate (xyz 0 0 0))
@@
       (net 63 "Net-(D42-Pad2)") (pinfunction "2") (pintype "passive"))
   )
-  (footprint "keeblib:alps_sksn" (layer "F.Cu")
-    (at 152.1341 66.668 -90)
+  (footprint "kbd:ResetSW_1side" (layer "F.Cu")
+    (at 153.4575 66.668 -90)
     (property "Sheetfile" "File: cho-corne-ice.kicad_sch")
     (property "Sheetname" "")
     (attr through_hole)
-    (fp_text reference "RSW2" (at 0 -0.8154 -90) (layer "F.SilkS")
+    (fp_text reference "RSW2" (at 0 2.55 -90) (layer "F.SilkS") hide
+      (effects (font (size 1 1) (thickness 0.15)))
+    )
+    (fp_text value "SW_PUSH" (at 0 -2.55 -90) (layer "F.Fab")
       (effects (font (size 1 1) (thickness 0.15)))
     )
-    (fp_text value "SW_PUSH" (at 0 -0.5 -90) (layer "F.Fab") hide
+    (fp_text user "RESET" (at 0 0 -90) (layer "F.SilkS")
       (effects (font (size 1 1) (thickness 0.15)))
     )
-    (fp_line (start 2.55 -1.65) (end 2.55 0) (layer "B.Fab") (width 0.12))
-    (fp_line (start -2.55 0) (end -2.55 -1.65) (layer "B.Fab") (width 0.12))
-    (fp_line (start -2.55 -1.65) (end 2.55 -1.65) (layer "B.Fab") (width 0.12))
-    (pad "" smd rect locked (at -3.2 -0.85 270) (size 0.6 0.8) (layers "F.Cu" "F.Paste" "F.Mask"))
-    (pad "" smd rect locked (at 3.2 -0.85 270) (size 0.6 0.8) (layers "F.Cu" "F.Paste" "F.Mask"))
-    (pad "1" smd rect locked (at 2.275 -2.575 270) (size 1.45 1.05) (layers "F.Cu" "F.Paste" "F.Mask")
+    (fp_line (start -2.85 1.6) (end 2.85 1.6) (layer "F.SilkS") (width 0.15))
+    (fp_line (start 2.85 1.6) (end 2.85 1.35) (layer "F.SilkS") (width 0.15))
+    (fp_line (start -2.85 1.6) (end -2.85 1.35) (layer "F.SilkS") (width 0.15))
+    (fp_line (start -2.85 -1.6) (end -2.85 -1.35) (layer "F.SilkS") (width 0.15))
+    (fp_line (start 2.85 -1.6) (end 2.85 -1.35) (layer "F.SilkS") (width 0.15))
+    (fp_line (start -2.85 -1.6) (end 2.85 -1.6) (layer "F.SilkS") (width 0.15))
+    (pad "1" thru_hole circle locked (at 3.25 0 270) (size 2 2) (drill 1.3) (layers *.Cu "B.Mask")
       (net 65 "reset_r") (pinfunction "1") (pintype "passive"))
-    (pad "2" smd rect locked (at -2.275 -2.575 270) (size 1.45 1.05) (layers "F.Cu" "F.Paste" "F.Mask")
+    (pad "2" thru_hole circle locked (at -3.25 0 270) (size 2 2) (drill 1.3) (layers *.Cu "B.Mask")
       (net 73 "GNDA") (pinfunction "2") (pintype "passive"))
-    (model "C:/Users/cwiggins/Downloads/keyboards/keeblib.pretty/3d/3Dâéâfâï_SKSNL.STEP"
-      (offset (xyz 0 2 0))
+    (model "/Users/foostan/src/github.com/foostan/kbd/kicad-packages3D/kbd.3dshapes/tact-switch.step"
+      (offset (xyz 0 0 3.47))
       (scale (xyz 1 1 1))
       (rotate (xyz 0 0 0))
@@
   (gr_curve (pts (xy 67.043905 83.166629) (xy 66.950153 83.072818) (xy 66.822965 83.020103) (xy 66.690339 83.020073)) (layer "Edge.Cuts") (width 0.2))
   (gr_curve (pts (xy 115.2655 102.67) (xy 115.05207 102.605557) (xy 114.832837 102.562169) (xy 114.610944 102.54046)) (layer "Edge.Cuts") (width 0.2))
+  (gr_arc (start 144.9231 63.9756) (mid 144.9231 63.9756) (end 144.9231 63.9756) (layer "Edge.Cuts") (width 0.2))
   (gr_line (start 230.204661 83.028073) (end 236.3275 83.028073) (layer "Edge.Cuts") (width 0.2))
   (gr_line (start 285.204501 83.028073) (end 279.0775 83.028073) (layer "Edge.Cuts") (width 0.2))

Commit message: complete layout and traces
Parts:
- removed LED24: YS-SK6812MINI-E, kbd:YS-SK6812MINI-E
- RSW1, RSW2: footprint kbd:ResetSW_1side -> keeblib:alps_sksn
- U1, U2: footprint nice-nano-kicad:nice_nano -> kbd:ProMicro_v3.5
- moved RSW1 1.58 mm to (144.7, 67.2)
- moved RSW2 1.43 mm to (152.2, 67.3)
- moved D21 0.63 mm to (98.0, 88.1), turned to -90 degrees
- moved D41 0.57 mm to (199.7, 88.1), turned to -90 degrees
- moved D19 0.17 mm to (76.0, 88.8), turned to -90 degrees
- moved PSW1 0.06 mm to (134.7, 28.9)
- turned D1 to -90 degrees
- turned D10 to -90 degrees
- turned D11 to -90 degrees
- turned D12 to -90 degrees
- turned D13 to -90 degrees
- turned D14 to -90 degrees
- turned D15 to -90 degrees
- turned D16 to -90 degrees
- turned D17 to -90 degrees
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Connections:
- J1 pad 1: RAW -> Net-(PSW1-Pad2)
- J1 pad 2: Net-(J1-Pad2) -> GND
- J3 pad 1: RAW_r -> Net-(PSW2-Pad2)
- J3 pad 2: Net-(J3-Pad2) -> GNDA
- PSW1 pad 1: Net-(J1-Pad2) -> RAW
- PSW1 pad 2: GND -> Net-(PSW1-Pad2)
- PSW2 pad 1: Net-(J3-Pad2) -> RAW_r
- PSW2 pad 2: GNDA -> Net-(PSW2-Pad2)
- RSW2 pad 1: reset_r -> GNDA
- RSW2 pad 2: GNDA -> reset_r
Routing:
- net col0: track 0.00 -> 170.6 mm, vias 0 -> 5
- net col0_r: track 0.00 -> 170.3 mm, vias 0 -> 4
- net col1: track 0.00 -> 154.5 mm, vias 0 -> 5
- net col1_r: track 0.00 -> 145.0 mm, vias 0 -> 4
- net col3_r: track 0.00 -> 128.8 mm, vias 0 -> 6
- net col3: track 0.00 -> 128.5 mm, vias 0 -> 7
- net col2_r: track 0.00 -> 123.0 mm, vias 0 -> 4
- net col2: track 0.00 -> 122.0 mm, vias 0 -> 4
- net col4_r: track 0.00 -> 114.4 mm, vias 0 -> 6
- net col4: track 0.00 -> 110.9 mm, vias 0 -> 8
- net col5: track 0.00 -> 106.4 mm, vias 0 -> 10
- net GND: track 0.00 -> 97.1 mm, vias 0 -> 1
- net GNDA: track 0.00 -> 96.6 mm, vias 0 -> 1
- net col5_r: track 0.00 -> 85.2 mm, vias 0 -> 6
- net row3_r: track 0.00 -> 74.6 mm
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Other:
- outline, holes or cut-outs redrawn
