File: cho-corne-ice/pcb/cho-corne-ice.kicad_pcb (KiCad board)
At the start: 2 copper layers, 275.5 x 105.6 mm, 120 parts, among them J1 BAT, J2 nice!view, J3 BAT, J4 nice!view, SW1 SW_PUSH, SW10 SW_PUSH, SW11 SW_PUSH, SW12 SW_PUSH, SW13 SW_PUSH, SW14 SW_PUSH, SW15 SW_PUSH, SW16 SW_PUSH, SW17 SW_PUSH, SW18 SW_PUSH, SW19 SW_PUSH, SW2 SW_PUSH, SW20 SW_PUSH, SW21 SW_PUSH, SW22 SW_PUSH, SW23 SW_PUSH, SW24 SW_PUSH, SW25 SW_PUSH, SW26 SW_PUSH, SW27 SW_PUSH, SW28 SW_PUSH, SW29 SW_PUSH, SW3 SW_PUSH, SW30 SW_PUSH, SW31 SW_PUSH, SW32 SW_PUSH, SW33 SW_PUSH, SW34 SW_PUSH, SW35 SW_PUSH, SW36 SW_PUSH, SW37 SW_PUSH, SW38 SW_PUSH, SW39 SW_PUSH, SW4 SW_PUSH, SW40 SW_PUSH, SW41 SW_PUSH, SW42 SW_PUSH, SW5 SW_PUSH, SW6 SW_PUSH, SW7 SW_PUSH, SW8 SW_PUSH, SW9 SW_PUSH, U1 nice_nano, U2 nice_nano

Commit message: better labeling
Parts:
- PSW1, PSW2: value SW_SPDT -> POWER
- RSW1, RSW2: value SW_PUSH -> RST
- U1, U2: value nice_nano -> nice!nano; footprint kbd:ProMicro_v3.5 -> kbd:ProMicro_v3
Other:
- board text added: "Cho-Corne-Ice v0.2 PCB Designed by foostan/e3b0c442"
- board text added: "GND"
- board text added: "VCC"
- board text removed: "Corne Cherry v3.0.1 PCB Designed by foostan"
