File: cho-corne-ice/pcb/cho-corne-ice.kicad_sch (KiCad schematic)
At the start: 94 parts, among them J1 BAT, J2 nice!view, J3 BAT, J4 nice!view, SW1 SW_PUSH, SW10 SW_PUSH, SW11 SW_PUSH, SW12 SW_PUSH, SW13 SW_PUSH, SW14 SW_PUSH, SW15 SW_PUSH, SW16 SW_PUSH, SW17 SW_PUSH, SW18 SW_PUSH, SW19 SW_PUSH, SW2 SW_PUSH, SW20 SW_PUSH, SW21 SW_PUSH, SW22 SW_PUSH, SW23 SW_PUSH, SW24 SW_PUSH, SW25 SW_PUSH, SW26 SW_PUSH, SW27 SW_PUSH, SW28 SW_PUSH, SW29 SW_PUSH, SW3 SW_PUSH, SW30 SW_PUSH, SW31 SW_PUSH, SW32 SW_PUSH, SW33 SW_PUSH, SW34 SW_PUSH, SW35 SW_PUSH, SW36 SW_PUSH, SW37 SW_PUSH, SW38 SW_PUSH, SW39 SW_PUSH, SW4 SW_PUSH, SW40 SW_PUSH, SW41 SW_PUSH, SW42 SW_PUSH, SW5 SW_PUSH, SW6 SW_PUSH, SW7 SW_PUSH, SW8 SW_PUSH, SW9 SW_PUSH, U1 nice_nano, U2 nice_nano

Commit message: better labeling
Parts:
- U1, U2: footprint kbd:ProMicro_v3.5 -> kbd:ProMicro_v3
Other:
- company: foostan & e3b0c442 -> foostan/e3b0c442
Changed lines of the file:
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@@
   (title_block
     (title "Cho-Corne-Ice")
-    (date "2020-09-28")
-    (rev "3.0.1")
-    (company "foostan & e3b0c442")
+    (date "2022-11-18")
+    (rev "v0.2")
+    (company "foostan/e3b0c442")
   )
   (junction (at 157.48 64.77) (diameter 0) (color 0 0 0 0)
@@
       (effects (font (size 1.524 1.524)))
     )
-    (property "Footprint" "kbd:ProMicro_v3.5" (id 2) (at 72.39 107.95 90)
+    (property "Footprint" "kbd:ProMicro_v3" (id 2) (at 72.39 107.95 90)
       (effects (font (size 1.524 1.524)) hide)
     )
@@
       (effects (font (size 1.524 1.524)))
     )
-    (property "Footprint" "kbd:ProMicro_v3.5" (id 2) (at 74.93 226.06 90)
+    (property "Footprint" "kbd:ProMicro_v3" (id 2) (at 74.93 226.06 90)
       (effects (font (size 1.524 1.524)) hide)
     )
@@
     )
     (path "/ce793b9a-acc0-4fe7-8442-3462bee6f436"
-      (reference "U1") (unit 1) (value "nice_nano") (footprint "kbd:ProMicro_v3.5")
+      (reference "U1") (unit 1) (value "nice_nano") (footprint "kbd:ProMicro_v3")
     )
     (path "/da44033a-0246-4bfa-820f-af5b696ffd2c"
-      (reference "U2") (unit 1) (value "nice_nano") (footprint "kbd:ProMicro_v3.5")
-    )
-  )
+      (reference "U2") (unit 1) (value "nice_nano") (footprint "kbd:ProMicro_v3")
+    )
+  )
